File: kicad/busy-board.kicad_pcb (KiCad board)
At the start: 4 copper layers, 137.2 x 180.3 mm, 249 parts, among them J201 JST PH 2P, J202 USB_C_Receptacle_PowerOnly_6P, Q201 AO3401A, Q301 MMBT3904, Q302 MMBT3904, Q303 MMBT3904, Q304 MMBT3904, Q305 MMBT3904, Q306 MMBT3904, Q307 MMBT3904, Q308 MMBT3904, Q309 MMBT3904, Q401 MMBT3904, Q501 MMBT3904, Q502 MMBT3904, Q503 MMBT3904, Q504 MMBT3904, Q505 MMBT3904, Q506 MMBT3904, Q507 MMBT3904, Q508 MMBT3904, Q509 MMBT3904, Q510 MMBT3904, Q601 MMBT3904, Q602 MMBT3904, Q603 MMBT3904, Q604 MMBT3904, Q605 MMBT3904, Q606 MMBT3904, Q607 MMBT3904, SW101 MAN_CNT, SW102 CLK_SELECT, SW201 SW_DIP_x04, SW202 SW_SPDT, SW301 SW Red, SW302 SW Orange, SW303 SW Green, SW304 SW White, SW305 SW Blue, SW306 SW Purple, SW401 DISP_SELECT, U101 LM393, U102 LM393, U103 4040, U104 LM393, U201 AMS1117-3.3, U202 TPD1E05U06DPY, U203 TPD1E05U06DPY, U204 TPS61040DBV, U205 TP4056-42-ESOP8, U401 4028, U402 4510, U403 4511, U501 74HC08D, U502 74HC08D, U503 74HC08D, U601 74HC08D, U602 74HC08D

Commit message: Fix v1 issues
- Change BJT to MOSFET for LED control: voltage drop on PWM
- Change voltage switch to PWM switch for 7-seg and bar control
- Change LDO to limit drop-out with battery
- Decrease resistor on Purple LED to increase luminosity
Parts:
- Q301, Q302, Q303, Q304, Q305, Q306, Q307, Q308, Q309, Q401, Q501, Q502, Q503, Q504, Q505, Q506, Q507, Q508, Q509, Q510, Q601, Q602, Q603, Q604, Q605, Q606, Q607: value MMBT3904 -> AO3400A
- R319: value 390 -> 360
- R320: value 360 -> 300
- U201: value AMS1117-3.3 -> XC6206P332MR; footprint Package_TO_SOT_SMD:SOT-223-3_TabPin2 -> Package_TO_SOT_SMD:SOT-23-3
- moved TP201 45.4 mm to (17.8, 61.0)
- moved J201 6.22 mm to (31.0, 19.4), turned to 90 degrees
- moved U201 3.01 mm to (36.7, 39.1), turned to 90 degrees
- moved R210 1.44 mm to (49.1, 29.3)
- moved R211 1.44 mm to (49.1, 26.4)
- moved R212 1.44 mm to (49.1, 23.4)
- moved R209 1.44 mm to (49.1, 32.3)
- moved SW201 1.44 mm to (46.7, 31.6)
- moved R202 0.28 mm to (34.1, 24.1)
- moved C206 0.28 mm to (34.1, 25.6)
- moved C205 0.28 mm to (34.1, 22.6)
Connections:
- C402 pad 1: /Counter/PWR_LED_BAR -> +3V3
- C403 pad 1: /Counter/PWR_LED_SEG -> +3V3
- J201 pad 1: Net-(J201-Pin_1) -> GND
- J201 pad 2: GND -> Net-(J201-Pin_2)
- R413 pad 1: /Counter/PWR_LED_COUNTER -> +3V3
- R414 pad 2: /Counter/PWR_LED_SEG -> +3V3
- SW102 pad 6: /CLK_CNT -> unconnected-(SW102-Pad6)
- SW102 pad 7: (no net) -> unconnected-(SW102-Pad7)
- SW102 pad 8: (no net) -> /CLK_CNT
- SW202 pad 2: Net-(J201-Pin_1) -> Net-(J201-Pin_2)
- SW401 pad 1: /Counter/PWR_LED_COUNTER -> /Counter/PWM_LED_COUNTER
- SW401 pad 2: /Counter/PWR_LED_BAR -> /Counter/PWM_LED_BAR
- SW401 pad 3: +3V3 -> /LED_PWM
- SW401 pad 4: /Counter/PWR_LED_SEG -> /Counter/PWM_LED_SEG
- U401 pad 16: /Counter/PWR_LED_BAR -> +3V3
- U403 pad 16: /Counter/PWR_LED_SEG -> +3V3
- U501 pad 10: /LED_PWM -> /Counter/PWM_LED_BAR
- U501 pad 13: /LED_PWM -> /Counter/PWM_LED_BAR
- U501 pad 2: /LED_PWM -> /Counter/PWM_LED_BAR
- U501 pad 5: /LED_PWM -> /Counter/PWM_LED_BAR
- U502 pad 10: /LED_PWM -> /Counter/PWM_LED_BAR
- U502 pad 13: /LED_PWM -> /Counter/PWM_LED_BAR
- U502 pad 2: /LED_PWM -> /Counter/PWM_LED_BAR
- U502 pad 5: /LED_PWM -> /Counter/PWM_LED_BAR
- U503 pad 10: /LED_PWM -> /Counter/PWM_LED_BAR
- U503 pad 13: /LED_PWM -> /Counter/PWM_LED_BAR
- U503 pad 5: /LED_PWM -> /Counter/PWM_LED_COUNTER
- U601 pad 10: /LED_PWM -> /Counter/PWM_LED_SEG
- U601 pad 13: /LED_PWM -> /Counter/PWM_LED_SEG
- U601 pad 2: /LED_PWM -> /Counter/PWM_LED_SEG
- U601 pad 5: /LED_PWM -> /Counter/PWM_LED_SEG
- U602 pad 10: /LED_PWM -> /Counter/PWM_LED_SEG
- U602 pad 13: /LED_PWM -> /Counter/PWM_LED_SEG
- U602 pad 5: /LED_PWM -> /Counter/PWM_LED_SEG
Routing:
- net /LED_PWM: track 444.5 -> 223.4 mm, vias 5 -> 1
- net /Counter/PWM_LED_SEG: track 0.00 -> 145.3 mm, vias 0 -> 2
- net /Counter/PWR_LED_SEG: track 101.1 -> 0.00 mm, vias 1 -> 0
- net /Counter/PWM_LED_BAR: track 0.00 -> 95.7 mm, vias 0 -> 3
- net /Counter/PWR_LED_COUNTER: track 68.6 -> 0.00 mm, vias 1 -> 0
- net /Counter/PWM_LED_COUNTER: track 0.00 -> 61.5 mm
- net /Counter/PWR_LED_BAR: track 50.4 -> 0.00 mm, vias 1 -> 0
- net Net-(J201-Pin_2): track 0.00 -> 14.6 mm
- net /CLK_CNT: track 38.0 -> 46.4 mm
- net +3V3: track 841.8 -> 850.1 mm, vias 46 -> 49
- net Net-(J201-Pin_1): track 7.68 -> 0.00 mm
- net +BATT: track 41.3 -> 38.9 mm
- net /CLK_4: track 163.2 -> 162.3 mm
- net Net-(U205-PROG): track 15.5 -> 16.2 mm
- net GND: vias 862 -> 855
- added copper zone on F.Cu, net Net-(J201-Pin_2)
- removed copper zone on In2.Cu, net /Counter/PWR_LED_BAR
- removed copper zone on In2.Cu, net /Counter/PWR_LED_COUNTER
- removed copper zone on In2.Cu, net /Counter/PWR_LED_SEG
- removed copper zone on F.Cu, net Net-(J201-Pin_1)
Other:
- board text added: "+ -"
- board text added: "Busy Board v1.1.0"
- board text removed: "Busy Board v1.0.0"
