File: kicad/counter.kicad_sch (KiCad schematic)
At the start: 32 parts, among them Q401 MMBT3904, SW401 DISP_SELECT, U401 4028, U402 4510, U403 4511

Commit message: Fix v1 issues
- Change BJT to MOSFET for LED control: voltage drop on PWM
- Change voltage switch to PWM switch for 7-seg and bar control
- Change LDO to limit drop-out with battery
- Decrease resistor on Purple LED to increase luminosity
Parts:
- removed Q401: MMBT3904, Package_TO_SOT_SMD:SOT-23, symbol Transistor_BJT:MMBT3904
- added Q401: AO3400A, Package_TO_SOT_SMD:SOT-23, symbol Transistor_FET:AO3400A
Connections:
- net +3V3: now also C402.1, C403.1, R413.1, R414.2, U401.16 (VDD), U403.16 (Vdd); no longer SW401.3
- net GND: now also Q401.2 (S)
- net PWM: now also SW401.3
- net at D401.1 (K): now also Q401.3 (D)
- net at R422.2: now also Q401.1 (G)
- removed net PWR_LED_BAR: C402.1, SW401.2, U401.16 (VDD)
- net PWR_LED_COUNTER renamed PWM_LED_COUNTER
- net PWM_LED_COUNTER: no longer R413.1
- removed net PWR_LED_SEG: C403.1, R414.2, SW401.4, U403.16 (Vdd)
- new net PWM_LED_BAR: SW401.2
- new net PWM_LED_SEG: SW401.4
Other:
- sheet Display Bar ports: added PWM_BAR, PWM_CNT; removed PWM
