File: kicad/display_7seg.kicad_sch (KiCad schematic)
At the start: 46 parts, among them Q601 MMBT3904, Q602 MMBT3904, Q603 MMBT3904, Q604 MMBT3904, Q605 MMBT3904, Q606 MMBT3904, Q607 MMBT3904, U601 74HC08D, U602 74HC08D

Commit message: Fix v1 issues
- Change BJT to MOSFET for LED control: voltage drop on PWM
- Change voltage switch to PWM switch for 7-seg and bar control
- Change LDO to limit drop-out with battery
- Decrease resistor on Purple LED to increase luminosity
Parts:
- removed Q601, Q602, Q603, Q604, Q605, Q606, Q607: MMBT3904, Package_TO_SOT_SMD:SOT-23, symbol Transistor_BJT:MMBT3904
- added Q601, Q602, Q603, Q604, Q605, Q606, Q607: AO3400A, Package_TO_SOT_SMD:SOT-23, symbol Transistor_FET:AO3400A
Connections:
- net GND: now also Q601.2 (S), Q602.2 (S), Q603.2 (S), Q604.2 (S), Q605.2 (S), Q606.2 (S), Q607.2 (S)
- net at R620.1: now also Q606.1 (G)
- net at D603.1 (K), D604.1 (K): now also Q602.3 (D)
- net at D609.1 (K), D610.1 (K): now also Q605.3 (D)
- net at D605.1 (K), D606.1 (K): now also Q603.3 (D)
- net at D611.1 (K), D612.1 (K): now also Q606.3 (D)
- net at R621.1: now also Q607.1 (G)
- net at D613.1 (K), D614.1 (K): now also Q607.3 (D)
- net at R617.1: now also Q603.1 (G)
- net at D607.1 (K), D608.1 (K): now also Q604.3 (D)
- net at D601.1 (K), D602.1 (K): now also Q601.3 (D)
- net at R615.1: now also Q601.1 (G)
- net at R618.1: now also Q604.1 (G)
- net at R619.1: now also Q605.1 (G)
- net at R616.1: now also Q602.1 (G)
