File: kicad/display_bar.kicad_sch (KiCad schematic)
At the start: 46 parts, among them Q501 MMBT3904, Q502 MMBT3904, Q503 MMBT3904, Q504 MMBT3904, Q505 MMBT3904, Q506 MMBT3904, Q507 MMBT3904, Q508 MMBT3904, Q509 MMBT3904, Q510 MMBT3904, U501 74HC08D, U502 74HC08D, U503 74HC08D

Commit message: Fix v1 issues
- Change BJT to MOSFET for LED control: voltage drop on PWM
- Change voltage switch to PWM switch for 7-seg and bar control
- Change LDO to limit drop-out with battery
- Decrease resistor on Purple LED to increase luminosity
Parts:
- removed Q501, Q502, Q503, Q504, Q505, Q506, Q507, Q508, Q509, Q510: MMBT3904, Package_TO_SOT_SMD:SOT-23, symbol Transistor_BJT:MMBT3904
- added Q501, Q502, Q503, Q504, Q505, Q506, Q507, Q508, Q509, Q510: AO3400A, Package_TO_SOT_SMD:SOT-23, symbol Transistor_FET:AO3400A
Connections:
- net GND: now also Q501.2 (S), Q502.2 (S), Q503.2 (S), Q504.2 (S), Q505.2 (S), Q506.2 (S), Q507.2 (S), Q508.2 (S), Q509.2 (S), Q510.2 (S)
- net at R514.1: now also Q504.1 (G)
- net at D504.1 (K): now also Q504.3 (D)
- net at R518.1: now also Q508.1 (G)
- net at D502.1 (K): now also Q502.3 (D)
- net at D510.1 (K): now also Q510.3 (D)
- net at D509.1 (K): now also Q509.3 (D)
- net at R512.1: now also Q502.1 (G)
- net at R516.1: now also Q506.1 (G)
- net at D503.1 (K): now also Q503.3 (D)
- net at D507.1 (K): now also Q507.3 (D)
- net at D508.1 (K): now also Q508.3 (D)
- net at R519.1: now also Q509.1 (G)
- net at R515.1: now also Q505.1 (G)
- net at D506.1 (K): now also Q506.3 (D)
- net at R520.1: now also Q510.1 (G)
- net at D501.1 (K): now also Q501.3 (D)
- net at R513.1: now also Q503.1 (G)
- net at D505.1 (K): now also Q505.3 (D)
- net at R511.1: now also Q501.1 (G)
- net at R517.1: now also Q507.1 (G)
- net PWM renamed PWM_BAR
- net PWM_BAR: no longer U503.5 (2B)
- new net PWM_CNT: U503.5 (2B)
