File: kicad/led.kicad_sch (KiCad schematic)
At the start: 48 parts, among them Q301 MMBT3904, Q302 MMBT3904, Q303 MMBT3904, Q304 MMBT3904, Q305 MMBT3904, Q306 MMBT3904, Q307 MMBT3904, Q308 MMBT3904, Q309 MMBT3904, SW301 SW Red, SW302 SW Orange, SW303 SW Green, SW304 SW White, SW305 SW Blue, SW306 SW Purple

Commit message: Fix v1 issues
- Change BJT to MOSFET for LED control: voltage drop on PWM
- Change voltage switch to PWM switch for 7-seg and bar control
- Change LDO to limit drop-out with battery
- Decrease resistor on Purple LED to increase luminosity
Parts:
- removed Q301, Q302, Q303, Q304, Q305, Q306, Q307, Q308, Q309: MMBT3904, Package_TO_SOT_SMD:SOT-23, symbol Transistor_BJT:MMBT3904
- added Q301, Q302, Q303, Q304, Q305, Q306, Q307, Q308, Q309: AO3400A, Package_TO_SOT_SMD:SOT-23, symbol Transistor_FET:AO3400A
- R319: value 390 -> 360; LCSC Part # C23151 -> C25194; MFR Part # 0603WAF3900T5E -> 0603WAF3600T5E
- R320: value 360 -> 300; LCSC Part # C25194 -> C23025; MFR Part # 0603WAF3600T5E -> 0603WAF3000T5E
Connections:
- net GND: now also Q301.2 (S), Q302.2 (S), Q303.2 (S), Q304.2 (S), Q305.2 (S), Q306.2 (S), Q307.2 (S), Q308.2 (S), Q309.2 (S)
- net at R313.2, R317.2: now also Q306.1 (G)
- net at R304.2: now also Q301.1 (G)
- net at D301.1 (K): now also Q301.3 (D)
- net at R321.2, R323.2: now also Q308.1 (G)
- net at D306.1 (K): now also Q306.3 (D)
- net at R306.2: now also Q303.1 (G)
- net at D303.1 (K): now also Q303.3 (D)
- net at D308.1 (K): now also Q308.3 (D)
- net at R311.2, R315.2: now also Q304.1 (G)
- net at R314.2, R318.2: now also Q307.1 (G)
- net at D307.1 (K): now also Q307.3 (D)
- net at D304.1 (K): now also Q304.3 (D)
- net at R312.2, R316.2: now also Q305.1 (G)
- net at R305.2: now also Q302.1 (G)
- net at D305.1 (K): now also Q305.3 (D)
- net at R322.2, R324.2: now also Q309.1 (G)
- net at D302.1 (K): now also Q302.3 (D)
- net at D309.1 (K): now also Q309.3 (D)
