File: kicad/power.kicad_sch (KiCad schematic)
At the start: 37 parts, among them J201 JST PH 2P, J202 USB_C_Receptacle_PowerOnly_6P, Q201 AO3401A, SW201 SW_DIP_x04, SW202 SW_SPDT, U201 AMS1117-3.3, U202 TPD1E05U06DPY, U203 TPD1E05U06DPY, U204 TPS61040DBV, U205 TP4056-42-ESOP8

Commit message: Fix v1 issues
- Change BJT to MOSFET for LED control: voltage drop on PWM
- Change voltage switch to PWM switch for 7-seg and bar control
- Change LDO to limit drop-out with battery
- Decrease resistor on Purple LED to increase luminosity
Parts:
- removed U201: AMS1117-3.3, Package_TO_SOT_SMD:SOT-223-3_TabPin2, symbol Regulator_Linear:AMS1117-3.3
- added U201: XC6206P332MR, Package_TO_SOT_SMD:SOT-23-3, symbol Regulator_Linear:XC6206PxxxMR
Connections:
- net +3V3: now also U201.2 (VO)
- net +BATT: now also U201.3 (VI)
- net GND: now also J201.1 (Pin_1), U201.1 (GND); no longer J201.2 (Pin_2)
- net at SW202.2 (B): now also J201.2 (Pin_2); no longer J201.1 (Pin_1)
Other:
- moved on the sheet: J201
Changed lines of the file:
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@@
 	(title_block
 		(title "Busy Board")
-		(date "2026-08-08")
-		(rev "1.0.0")
+		(date "2026-09-25")
+		(rev "1.1.0")
 	)
 	(text "RPROG= IBAT\n30k   =   50mA\n20k   =   70mA\n10k   =  130mA *\n5k    =  250mA\n4k    =  300mA *\n3k    =  400mA\n2k    =  580mA *\n1.6k  =  690mA\n1.4k  =  780mA\n1.2k  =  900mA *\n1.1k  = 1000mA"
@@
 	(wire
 		(pts
+			(xy 121.92 30.48) (xy 124.46 30.48)
+		)
+		(stroke
+			(width 0)
+			(type default)
+		)
+	)
+	(wire
+		(pts
 			(xy 241.3 81.28) (xy 241.3 82.55)
 		)
@@
 	(wire
 		(pts
-			(xy 121.92 30.48) (xy 124.46 30.48)
-		)
-		(stroke
-			(width 0)
-			(type default)
-		)
-	)
-	(wire
-		(pts
 			(xy 78.74 184.15) (xy 78.74 185.42)
 		)
@@
 	(symbol
 		(lib_id "Connector_Generic:Conn_01x02")
-		(at 116.84 30.48 0)
-		(mirror y)
+		(at 116.84 33.02 180)
 		(unit 1)
 		(exclude_from_sim no)
@@
 		(dnp no)
 		(property "Reference" "J201"
-			(at 116.84 39.37 0)
+			(at 116.84 24.13 0)
 			(effects
 				(font
@@
 		)
 		(property "Value" "JST PH 2P"
-			(at 116.84 36.83 0)
+			(at 116.84 26.67 0)
 			(effects
 				(font
@@
 		)
 		(property "Footprint" "Connector_JST:JST_PH_S2B-PH-K_1x02_P2.00mm_Horizontal"
-			(at 116.84 30.48 0)
+			(at 116.84 33.02 0)
 			(effects
 				(font
@@
 		)
 		(property "Datasheet" "https://jlcpcb.com/api/file/downloadByFileSystemAccessId/8587713913773568000"
-			(at 116.84 30.48 0)
+			(at 116.84 33.02 0)
 			(effects
 				(font
@@
 		)
 		(property "Description" "Generic connector, single row, 01x02, script generated (kicad-library-utils/schlib/autogen/connector/)"
-			(at 116.84 30.48 0)
+			(at 116.84 33.02 0)
 			(effects
 				(font
@@
 		)
 		(property "LCSC Part #" "C173752"
-			(at 116.84 30.48 0)
+			(at 116.84 33.02 0)
 			(effects
 				(font
@@
 		)
 		(property "Manufacturer" "JST"
-			(at 116.84 30.48 0)
+			(at 116.84 33.02 0)
 			(effects
 				(font
@@
 		)
 		(property "MFR Part #" "S2B-PH-K-S(LF)(SN)"
-			(at 116.84 30.48 0)
+			(at 116.84 33.02 0)
 			(effects
 				(font
@@
 		)
 		(property "Sim.Library" ""
-			(at 116.84 30.48 0)
+			(at 116.84 33.02 0)
 			(effects
 				(font
@@
 		)
 		(property "Sim.Name" ""
-			(at 116.84 30.48 0)
+			(at 116.84 33.02 0)
 			(effects
 				(font
@@
 		)
 		(property "Sim.Params" ""
-			(at 116.84 30.48 0)
+			(at 116.84 33.02 0)
 			(effects
 				(font
@@
 	)
 	(symbol
+		(lib_id "Regulator_Linear:XC6206PxxxMR")
+		(at 231.14 30.48 0)
+		(unit 1)
+		(exclude_from_sim no)
+		(in_bom yes)
+		(on_board yes)
+		(dnp no)
+		(fields_autoplaced yes)
+		(property "Reference" "U201"
+			(at 231.14 24.13 0)
+			(effects
+				(font
+					(size 1.27 1.27)
+				)
+			)
+		)
+		(property "Value" "XC6206P332MR"
+			(at 231.14 26.67 0)
+			(effects
+				(font
+					(size 1.27 1.27)
+				)
+			)
+		)
+		(property "Footprint" "Package_TO_SOT_SMD:SOT-23-3"
+			(at 231.14 24.765 0)
+			(effects
+				(font
+					(size 1.27 1.27)
+					(italic yes)
+				)
+				(hide yes)
+			)
+		)
+		(property "Datasheet" "https://www.torexsemi.com/file/xc6206/XC6206.pdf"
+			(at 231.14 30.48 0)
+			(effects
+				(font
+					(size 1.27 1.27)
+				)
+				(hide yes)
+			)
+		)
+		(property "Description" "Positive 60-250mA Low Dropout Regulator, Fixed Output, SOT-23"
+			(at 231.14 30.48 0)
+			(effects
+				(font
+					(size 1.27 1.27)
+				)
+				(hide yes)
+			)
+		)
+		(property "LCSC Part #" "C5446"
+			(at 231.14 30.48 0)
+			(effects
+				(font
+					(size 1.27 1.27)
+				)
+				(hide yes)
+			)
+		)
+		(property "Manufacturer" "Torex Semicon"
+			(at 231.14 30.48 0)
+			(effects
+				(font
+					(size 1.27 1.27)
+				)
+				(hide yes)
+			)
+		)
+		(property "MFR Part #" "XC6206P332MR-G"
+			(at 231.14 30.48 0)
+			(effects
+				(font
+					(size 1.27 1.27)
+				)
+				(hide yes)
+			)
+		)
+		(pin "2"
+		)
+		(pin "3"
+		)
+		(pin "1"
+		)
+		(instances
+			(project "busy-board"
+				(path "/0502a6a9-5fe6-43a5-b6f7-3b5176fd87b6/94e5aaad-7bc2-4272-9b41-78f7bb3daed3"
+					(reference "U201")
+					(unit 1)
+				)
+			)
+		)
+	)
+	(symbol
 		(lib_id "Power_Protection:TPD1E05U06DPY")
 		(at 41.91 78.74 270)
@@
 					(unit 1)
 				)
-			)
-		)
-	)
-	(symbol
-		(lib_id "Regulator_Linear:AMS1117-3.3")
-		(at 231.14 30.48 0)
-		(unit 1)
-		(exclude_from_sim no)
-		(in_bom yes)
-		(on_board yes)
-		(dnp no)
-		(fields_autoplaced yes)
-		(property "Reference" "U201"
-			(at 231.14 24.13 0)
-			(effects
-				(font
-					(size 1.27 1.27)
-				)
-			)
-		)
-		(property "Value" "AMS1117-3.3"
-			(at 231.14 26.67 0)
-			(effects
-				(font
-					(size 1.27 1.27)
-				)
-			)
-		)
-		(property "Footprint" "Package_TO_SOT_SMD:SOT-223-3_TabPin2"
-			(at 231.14 25.4 0)
-			(effects
-				(font
-					(size 1.27 1.27)
-				)
-				(hide yes)
-			)
-		)
-		(property "Datasheet" "http://www.advanced-monolithic.com/pdf/ds1117.pdf"
-			(at 233.68 36.83 0)
-			(effects
-				(font
-					(size 1.27 1.27)
-				)
-				(hide yes)
-			)
-		)
-		(property "Description" "1A Low Dropout regulator, positive, 3.3V fixed output, SOT-223"
-			(at 231.14 30.48 0)
-			(effects
-				(font
-					(size 1.27 1.27)
-				)
-				(hide yes)
-			)
-		)
-		(property "LCSC Part #" "C6186"
-			(at 231.14 30.48 0)
-			(effects
-				(font
-					(size 1.27 1.27)
-				)
-				(hide yes)
-			)
-		)
-		(property "Manufacturer" "Advanced Monolithic Systems"
-			(at 231.14 30.48 0)
-			(effects
-				(font
-					(size 1.27 1.27)
-				)
-				(hide yes)
-			)
-		)
-		(property "MFR Part #" "AMS1117-3.3"
-			(at 231.14 30.48 0)
-			(effects
-				(font
-					(size 1.27 1.27)
-				)
-				(hide yes)
-			)
-		)
-		(property "Sim.Library" ""
-			(at 231.14 30.48 0)
-			(effects
-				(font
-					(size 1.27 1.27)
-				)
-				(hide yes)
-			)
-		)
-		(property "Sim.Name" ""
-			(at 231.14 30.48 0)
-			(effects
-				(font
-					(size 1.27 1.27)
-				)
-				(hide yes)
-			)
-		)
-		(property "Sim.Params" ""
-			(at 231.14 30.48 0)
-			(effects
-				(font
-					(size 1.27 1.27)
-				)
-				(hide yes)
-			)
-		)
-		(pin "1"
-		)
-		(pin "3"
-		)
-		(pin "2"
-		)
-		(instances
-			(project "busy-board"
-				(path "/0502a6a9-5fe6-43a5-b6f7-3b5176fd87b6/94e5aaad-7bc2-4272-9b41-78f7bb3daed3"
-					(reference "U201")
-					(unit 1)
-				)
